Commit message: fix xacro macro

File: urdf/sensors/magnetometer_snippets.xacro (robot description, xacro)
@@ -1,4 +1,4 @@
 <robot xmlns:xacro="http://www.ros.org/wiki/xacro">
-	<macro name="__ituauv_magnetometer_macro" params="namespace suffix parent_link topic mass update_rate
+	<xacro:macro name="__ituauv_magnetometer_macro" params="namespace suffix parent_link topic mass update_rate
 mag_intensity noise_xy noise_z turn_on_bias noise_amplitude
 *inertia *origin">
@@ -77,4 +77,4 @@
 			</plugin>
 		</gazebo>
-	</macro>
+	</xacro:macro>
 </robot>
