Commit message: fix

File: urdf/sensors/imu_snippets.xacro (robot description, xacro)
@@ -10,9 +10,9 @@
 			<xacro:insert_block name="origin" />
 			<!-- TODO: Add mesh file -->
-			<!-- <visual>
-				<geometry>
+			<visual>
+				<!-- <geometry>
 					<mesh filename="file://$(find ituauv_uuv_descriptions)/meshes/sensors/ping_sonar/ping_sonar.dae" scale="0.1 0.1 0.1" />
-				</geometry>
-			</visual> -->
+				</geometry> -->
+			</visual>
 		</xacro:__ituauv_imu_macro>
 		<xacro:__ituauv_magnetometer_macro

Commit message: seperate mag and imu

File: urdf/sensors/imu_snippets.xacro (robot description, xacro)
@@ -7,5 +7,22 @@
 	-->
 	<xacro:macro name="xsens_mti_g710" params="namespace topic topic_mag parent_link *origin">
-		<xacro:__ituauv_imu_macro namespace="${namespace}" imu_suffix="" parent_link="${parent_link}" imu_topic="${topic}" mass_imu_sensor="0.015" gyroscope_noise_density="0.0002514074" gyroscope_random_walk="0.000038785" gyroscope_bias_correlation_time="1000.0" gyroscope_turn_on_bias_sigma="0.0087" accelerometer_noise_density="0.00104347826" accelerometer_random_walk="0.006" accelerometer_bias_correlation_time="300.0" accelerometer_turn_on_bias_sigma="0.1960" orientation_noise="0.05" enable_local_ned_frame="false" reference_frame="world" update_rate="80">
+		<xacro:__ituauv_imu_macro
+			namespace="${namespace}"
+			imu_suffix=""
+			parent_link="${parent_link}"
+			imu_topic="${topic}"
+			mass_imu_sensor="0.015"
+			gyroscope_noise_density="0.0002514074"
+			gyroscope_random_walk="0.000038785"
+			gyroscope_bias_correlation_time="1000.0"
+			gyroscope_turn_on_bias_sigma="0.0087"
+			accelerometer_noise_density="0.00104347826"
+			accelerometer_random_walk="0.006"
+			accelerometer_bias_correlation_time="300.0"
+			accelerometer_turn_on_bias_sigma="0.1960"
+			orientation_noise="0.05"
+			enable_local_ned_frame="false"
+			reference_frame="world"
+			update_rate="80">
 			<inertia ixx="0.00001" ixy="0.0" ixz="0.0" iyy="0.00001" iyz="0.0" izz="0.00001" />
 			<xacro:insert_block name="origin" />
@@ -17,19 +34,4 @@
 			</visual>
 		</xacro:__ituauv_imu_macro>
-		<xacro:__ituauv_magnetometer_macro
-			namespace="${namespace}"
-			suffix=""
-			parent_link="${parent_link}"
-			topic="${topic_mag}"
-			mass="0.015"
-			update_rate="80"
-			mag_intensity="65.0"
-			noise_xy="1.0"
-			noise_z="1.4"
-			noise_amplitude="0.1"
-			turn_on_bias="2.0">
-			<inertia ixx="0.00001" ixy="0.0" ixz="0.0" iyy="0.00001" iyz="0.0" izz="0.00001" />
-			<origin xyz="0 0 0" rpy="0 0 0" />
-		</xacro:__ituauv_magnetometer_macro>
 	</xacro:macro>
 	<!-- Macro to add an IMU. -->

File: urdf/sensors/magnetometer_snippets.xacro (robot description, xacro)
@@ -1,4 +1,21 @@
 <?xml version="1.0"?>
 <robot xmlns:xacro="http://www.ros.org/wiki/xacro">
+	<xacro:macro name="xsens_mti_g710_mag" params="namespace topic parent_link *origin">
+		<xacro:__ituauv_magnetometer_macro
+			namespace="${namespace}"
+			suffix=""
+			parent_link="${parent_link}"
+			topic="${topic}"
+			mass="0.015"
+			update_rate="80"
+			mag_intensity="65.0"
+			noise_xy="1.0"
+			noise_z="1.4"
+			noise_amplitude="0.1"
+			turn_on_bias="2.0">
+			<inertia ixx="0.00001" ixy="0.0" ixz="0.0" iyy="0.00001" iyz="0.0" izz="0.00001" />
+			<origin xyz="0 0 0" rpy="0 0 0" />
+		</xacro:__ituauv_magnetometer_macro>
+	</xacro:macro>
 	<xacro:macro name="__ituauv_magnetometer_macro" params="namespace suffix parent_link topic mass update_rate
 mag_intensity noise_xy noise_z turn_on_bias noise_amplitude
